File: opusdiscovery.kicad_sch (KiCad schematic)
At the start: 61 parts, among them IC1 WD1772, IC11 GAL22V10, IC12 L7805, IC2 AT28C256, IC3 6264, IC4 GAL22V10, IC5 74LS06, IC9 74LS00, J1 ZX_Spectrum_Connector_GENERIC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, J2 Conn_02x17_Odd_Even, J3 Conn_02x13_Odd_Even, J4 DB9_Male, J5 DB25_Female_MountingHoles, SW2 SW_DPST_x2, SW3 SW_DIP_x03, U1 74LS73, U10 74LS38, U2 74LS139, U3 6821, Y1 8.000Mhz

Commit message: update gal equations
Other:
- note added: "CX_CK = !MREQ & RFSH;"
- note added: "CX_J = A6 & A8 & U8B_4;"
- note added: "CX_K = !(A6 & A8) & U8B_4;"
- note added: "CX_U6A_A1= CX_U12B_6 = !A15 # !A14 # RFSH # !MREQ"
- note added: "U8A_1 = !(U9B_6 # U9C_8 # U9D_11);"
- note added: "U8B_4 = U8A_1 & !A11 & A3 & !A13 & U12A_5 & CX_U12B_6 & !A4 & !M1 ;"
- note added: "U9B_6 = (A8 & !A9) # (!A8 & A9); U9C_8 = (A9 & !A10) # (!A9 & A10); U9D_11 = (A10 & !A12) # (!A10 & A12);"
Changed lines of the file:
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@@
     (stroke (width 0) (type solid) (color 0 0 0 0))
+  )
+  (text "U9B_6 = (A8 & !A9) # (!A8 & A9);\nU9C_8 = (A9 & !A10) # (!A9 & A10);\nU9D_11 = (A10 & !A12) # (!A10 & A12);"
+    (at 16.51 232.41 0)
+    (effects (font (size 1.27 1.27)) (justify left bottom))
+  )
+  (text "U8A_1 = !(U9B_6 # U9C_8 # U9D_11);" (at 16.51 236.22 0)
+    (effects (font (size 1.27 1.27)) (justify left bottom))
+  )
+  (text "U8B_4 = U8A_1 & !A11 & A3 & !A13 & U12A_5 & CX_U12B_6 & !A4 & !M1 ;"
+    (at 16.51 238.76 0)
+    (effects (font (size 1.27 1.27)) (justify left bottom))
+  )
+  (text "CX_J = A6 & A8 & U8B_4;" (at 31.75 215.9 0)
+    (effects (font (size 1.27 1.27)) (justify left bottom))
+  )
+  (text "CX_CK = !MREQ & RFSH;" (at 31.75 218.44 0)
+    (effects (font (size 1.27 1.27)) (justify left bottom))
+  )
+  (text "CX_K = !(A6 & A8) & U8B_4;" (at 31.75 220.98 0)
+    (effects (font (size 1.27 1.27)) (justify left bottom))
+  )
+  (text "CX_U6A_A1= CX_U12B_6 = !A15 # !A14 # RFSH # !MREQ" (at 116.84 195.58 180)
+    (effects (font (size 1.27 1.27)) (justify right bottom))
   )
   (text "Install D1 and D2  for 4K RAM upgrade.\ninstall only D1 (or a jumper) for original 2K Interface"
@@
     (effects (font (size 1.27 1.27)) (justify left bottom))
   )
+  (label "A14" (at 29.21 132.08 0)
+    (effects (font (size 1.27 1.27)) (justify left bottom))
+  )
+  (label "A15" (at 29.21 134.62 0)
+    (effects (font (size 1.27 1.27)) (justify left bottom))
+  )
+  (label "A13" (at 29.21 137.16 0)
+    (effects (font (size 1.27 1.27)) (justify left bottom))
+  )
+  (label "A12" (at 29.21 144.78 0)
+    (effects (font (size 1.27 1.27)) (justify left bottom))
+  )
+  (label "A11" (at 29.21 147.32 0)
+    (effects (font (size 1.27 1.27)) (justify left bottom))
+  )
+  (label "A6" (at 29.21 149.86 0)
+    (effects (font (size 1.27 1.27)) (justify left bottom))
+  )
+  (label "A5" (at 29.21 152.4 0)
+    (effects (font (size 1.27 1.27)) (justify left bottom))
+  )
+  (label "A4" (at 29.21 154.94 0)
+    (effects (font (size 1.27 1.27)) (justify left bottom))
+  )
+  (label "A3" (at 29.21 157.48 0)
+    (effects (font (size 1.27 1.27)) (justify left bottom))
+  )
   (label "MREQ" (at 30.48 139.7 0)
     (effects (font (size 1.27 1.27)) (justify left bottom))
   )
   (label "RFSH" (at 30.48 142.24 0)
+    (effects (font (size 1.27 1.27)) (justify left bottom))
+  )
+  (label "A9" (at 30.48 165.1 0)
+    (effects (font (size 1.27 1.27)) (justify left bottom))
+  )
+  (label "A10" (at 30.48 167.64 0)
     (effects (font (size 1.27 1.27)) (justify left bottom))
   )
@@
     (effects (font (size 1.27 1.27)) (justify left bottom))
   )
-  (label "A14" (at 31.75 132.08 0)
-    (effects (font (size 1.27 1.27)) (justify left bottom))
-  )
-  (label "A15" (at 31.75 134.62 0)
-    (effects (font (size 1.27 1.27)) (justify left bottom))
-  )
-  (label "A13" (at 31.75 137.16 0)
-    (effects (font (size 1.27 1.27)) (justify left bottom))
-  )
-  (label "A12" (at 33.02 144.78 0)
-    (effects (font (size 1.27 1.27)) (justify left bottom))
-  )
-  (label "A11" (at 33.02 147.32 0)
-    (effects (font (size 1.27 1.27)) (justify left bottom))
-  )
-  (label "A6" (at 33.02 149.86 0)
-    (effects (font (size 1.27 1.27)) (justify left bottom))
-  )
-  (label "A5" (at 33.02 152.4 0)
-    (effects (font (size 1.27 1.27)) (justify left bottom))
-  )
-  (label "A4" (at 33.02 154.94 0)
-    (effects (font (size 1.27 1.27)) (justify left bottom))
-  )
-  (label "A3" (at 33.02 157.48 0)
-    (effects (font (size 1.27 1.27)) (justify left bottom))
-  )
-  (label "A9" (at 33.02 165.1 0)
-    (effects (font (size 1.27 1.27)) (justify left bottom))
-  )
-  (label "A10" (at 33.02 167.64 0)
-    (effects (font (size 1.27 1.27)) (justify left bottom))
-  )
   (label "RD" (at 34.29 69.85 0)
     (effects (font (size 1.27 1.27)) (justify left bottom))
@@
     (effects (font (size 1.27 1.27)) (justify left bottom))
   )
+  (label "A8" (at 72.39 147.32 0)
+    (effects (font (size 1.27 1.27)) (justify left bottom))
+  )
+  (label "A7" (at 72.39 149.86 0)
+    (effects (font (size 1.27 1.27)) (justify left bottom))
+  )
   (label "M1" (at 74.295 144.78 0)
     (effects (font (size 1.27 1.27)) (justify left bottom))
   )
-  (label "A8" (at 74.295 147.32 0)
-    (effects (font (size 1.27 1.27)) (justify left bottom))
-  )
-  (label "A7" (at 74.295 149.86 0)
-    (effects (font (size 1.27 1.27)) (justify left bottom))
-  )
